Commit message: Update ur_macro.xacro to rename tool0 to tool0_ur and allow us to make our own tool0

File: ur_description/urdf/inc/ur_macro.xacro (robot description, xacro)
@@ -367,10 +367,10 @@
     </joint>
     <!-- ROS-Industrial 'tool0' frame: all-zeros tool frame -->
-    <link name="${prefix}tool0"/>
-    <joint name="${prefix}flange-tool0" type="fixed">
+    <link name="${prefix}tool0_ur"/>
+    <joint name="${prefix}flange-tool0_ur" type="fixed">
       <!-- default toolframe: X+ left, Y+ up, Z+ front -->
       <origin xyz="0 0 0" rpy="${pi/2.0} 0 ${pi/2.0}"/>
       <parent link="${prefix}flange"/>
-      <child link="${prefix}tool0"/>
+      <child link="${prefix}tool0_ur"/>
     </joint>
   </xacro:macro>
